Commit message: Update URDF: Convert absolute mesh paths to package-relative paths

File: src/ROAR_pkg/urdf/New_URDF.urdf (robot description, URDF)
Before this commit: robot New_URDF, 8 links, 7 joints
Links:
- link Link_1: geometry collision mesh filename=package://ROAR_pkg/meshes/Link_1.STL; visual mesh filename=package://ROAR_pkg/meshes/Link_1.STL
- link Link_2: geometry collision mesh filename=package://ROAR_pkg/meshes/Link_2.STL; visual mesh filename=package://ROAR_pkg/meshes/Link_2.STL
- link Link_3: geometry collision mesh filename=package://ROAR_pkg/meshes/Link_3.STL; visual mesh filename=package://ROAR_pkg/meshes/Link_3.STL
- link Link_4: geometry collision mesh filename=package://ROAR_pkg/meshes/Link_4.STL; visual mesh filename=package://ROAR_pkg/meshes/Link_4.STL
- link Link_5: geometry collision mesh filename=package://ROAR_pkg/meshes/Link_5.STL; visual mesh filename=package://ROAR_pkg/meshes/Link_5.STL
- link Link_EE: geometry collision mesh filename=package://ROAR_pkg/meshes/Link_EE.STL; visual mesh filename=package://ROAR_pkg/meshes/Link_EE.STL
- link base_link: geometry collision mesh filename=package://ROAR_pkg/meshes/base_link.STL; visual mesh filename=package://ROAR_pkg/meshes/base_link.STL

Commit message: refactor gazebo with rviz

File: src/ROAR_pkg/urdf/New_URDF.urdf (robot description, URDF)
Before this commit: robot New_URDF, 8 links, 7 joints
Joints:
- joint Joint_1: limit lower=-1.5708 upper=1.5708 effort=10.0 velocity=2.0 -> lower=-1.5808 upper=1.5808 effort=10.0 velocity=2.0
- joint Joint_2: limit lower=-2.4435 upper=0.0 effort=10.0 velocity=2.0 -> lower=-2.4535 upper=0.01 effort=10.0 velocity=2.0
- joint Joint_3: limit lower=-1.5708 upper=1.5708 effort=10.0 velocity=2.0 -> lower=-1.5808 upper=1.5808 effort=10.0 velocity=2.0
- joint Joint_4: limit lower=-1.5708 upper=1.5708 effort=10.0 velocity=2.0 -> lower=-1.5808 upper=1.5808 effort=10.0 velocity=2.0
- joint Joint_5: limit lower=-1.5708 upper=1.5708 effort=10.0 velocity=2.0 -> lower=-1.5808 upper=1.5808 effort=10.0 velocity=2.0
- joint Joint_EE: limit lower=-0.1173 upper=0.0 effort=10.0 velocity=1.0 -> lower=-0.1273 upper=0.01 effort=10.0 velocity=1.0
