Commit message: Add teleop scripts and README

File: src/ROAR_MoveIT/config/New_URDF.ros2_control.xacro (robot description, xacro)
@@ -2,5 +2,5 @@
 <robot xmlns:xacro="http://www.ros.org/wiki/xacro">
     <xacro:macro name="New_URDF_ros2_control" params="name initial_positions_file">
-        <xacro:property name="initial_positions" value="${xacro.load_yaml(initial_positions_file)['initial_positions']}"/>
+        <xacro:property name="initial_positions" value="${load_yaml(initial_positions_file)['initial_positions']}"/>
         <ros2_control name="${name}" type="system">
             <hardware>

File: src/ROAR_MoveIT/config/New_URDF.urdf.xacro (robot description, xacro)
@@ -5,5 +5,5 @@
     <xacro:include filename="$(find ROAR_pkg)/urdf/New_URDF.urdf" />
     <!-- Import control_xacro -->
-    <!--<xacro:include filename="New_URDF.ros2_control.xacro" />
-    <xacro:New_URDF_ros2_control name="FakeSystem" initial_positions_file="$(arg initial_positions_file)"/>-->
+    <xacro:include filename="New_URDF.ros2_control.xacro" />
+    <xacro:New_URDF_ros2_control name="FakeSystem" initial_positions_file="$(arg initial_positions_file)"/>
 </robot>
