Commit message: Align MoveIt/tooling EE frame to ee_link and refine tip offset

File: src/legacy_pkg/urdf/legacy.urdf (robot description, URDF)
Before this commit: robot legacy_pkg, 11 links, 10 joints
Links:
- added link ee_link
Joints:
- added joint ee_fixed_joint: type fixed, parent Link_5, child ee_link, origin xyz=0.0018 0.0064 0.0555 rpy=0 0 0
