Commit message: testing tool facing direction
Co-authored-by: Copilot <copilot@github.com>

File: src/sixdof_pkg/urdf/roar.urdf (robot description, URDF)
Before this commit: robot sixdof_pkg, 10 links, 9 joints
Joints:
- joint joint_0: limit lower=-0.017 upper=3.159 effort=150.0 velocity=1.0 -> lower=-1.5708 upper=1.5708 effort=150.0 velocity=1.0

Commit message: working gripper fr
Co-authored-by: Copilot <copilot@github.com>

File: src/sixdof_pkg/urdf/roar.urdf (robot description, URDF)
Before this commit: robot sixdof_pkg, 10 links, 9 joints
Joints:
- joint left_gripper: axis 0 0 1 -> 0 0 -1; origin xyz=0.0855 -0.0175 0.1025 rpy=-1.5708 -0.13911 1.5708 -> xyz=0.0165 -0.0175 0.1025 rpy=-1.5708 -0.13911 1.5708

Commit message: 6dof on rover
Co-authored-by: Copilot <copilot@github.com>

File: src/sixdof_pkg/urdf/roar.urdf (robot description, URDF)
Before this commit: robot sixdof_pkg, 10 links, 9 joints
Joints:
- joint joint_0: axis 0 0 1 -> 0 0 -1; origin xyz=0 0 0.12313 rpy=0 0 3.1416 -> xyz=-0.36681 -0.39666 0.030332 rpy=0 0 -1.5708
- joint world_to_base: origin xyz=0 0 0 rpy=0 0 0 -> xyz=0 0 0.5170493 rpy=0 0 0
