Commit message: rviz and gazebo done

File: src/sixdof_pkg/urdf/roar.urdf (robot description, URDF)
Before this commit: robot sixdof_pkg, 10 links, 9 joints
Joints:
- joint joint_5: origin xyz=-0.008596 -0.061393 0 rpy=1.7099 -1.5708 0 -> xyz=-0.008596 -0.061393 0 rpy=1.4317 -1.5708 0

Commit message: el3ab ya arm

File: src/sixdof_pkg/urdf/roar.urdf (robot description, URDF)
Before this commit: robot sixdof_pkg, 10 links, 9 joints
Joints:
- joint left_gripper: axis 0 0 1 -> 0 0 -1; limit lower=0.0 upper=0.2 effort=40.0 velocity=0.2 -> lower=-0.075 upper=0.0 effort=40.0 velocity=0.2
- joint right_gripper: limit lower=0.0 upper=0.2 effort=40.0 velocity=0.2 -> lower=0.0 upper=0.075 effort=40.0 velocity=0.2

Commit message: added storage poses

File: src/sixdof_pkg/urdf/roar.urdf (robot description, URDF)
Before this commit: robot sixdof_pkg, 10 links, 9 joints
Joints:
- joint joint_0: limit lower=-1.5708 upper=1.5708 effort=150.0 velocity=1.0 -> lower=-3.1416 upper=3.1416 effort=150.0 velocity=1.0
