Commit message: gripper works

File: src/sixdof_moveit/config/sixdof_pkg.urdf.xacro (robot description, xacro)
@@ -2,6 +2,9 @@
 <robot xmlns:xacro="http://www.ros.org/wiki/xacro" name="sixdof_pkg">
     <xacro:arg name="initial_positions_file" default="initial_positions.yaml" />
+    <xacro:arg name="use_mock_hardware" default="false" />
     <xacro:include filename="$(find sixdof_pkg)/urdf/roar.urdf" />
     <xacro:include filename="sixdof_pkg.ros2_control.xacro" />
-    <xacro:sixdof_pkg_ros2_control name="FakeSystem" initial_positions_file="$(arg initial_positions_file)"/>
+    <xacro:if value="$(arg use_mock_hardware)">
+        <xacro:sixdof_pkg_ros2_control name="FakeSystem" initial_positions_file="$(arg initial_positions_file)"/>
+    </xacro:if>
 </robot>

File: src/sixdof_pkg/urdf/roar.urdf (robot description, URDF)
Before this commit: robot sixdof_pkg, 10 links, 9 joints
Joints:
- joint left_gripper: axis 0 0 -1 -> 0 0 1; limit lower=-0.075 upper=0.0 effort=40.0 velocity=0.2 -> lower=0.0 upper=0.08 effort=40.0 velocity=0.2
- joint right_gripper: limit lower=0.0 upper=0.075 effort=40.0 velocity=0.2 -> lower=0.0 upper=0.08 effort=40.0 velocity=0.2

Commit message: fully functional interchangeable tips

File: src/sixdof_moveit/config/sixdof_pkg.urdf.xacro (robot description, xacro)
@@ -3,5 +3,5 @@
     <xacro:arg name="initial_positions_file" default="initial_positions.yaml" />
     <xacro:arg name="use_mock_hardware" default="false" />
-    <xacro:include filename="$(find sixdof_pkg)/urdf/roar.urdf" />
+    <xacro:include filename="$(find sixdof_pkg)/urdf/roar_variant.urdf.xacro" />
     <xacro:include filename="sixdof_pkg.ros2_control.xacro" />
     <xacro:if value="$(arg use_mock_hardware)">

File: src/sixdof_pkg/urdf/roar.urdf (robot description, URDF)
Before this commit: robot sixdof_pkg, 10 links, 9 joints
Links:
- added link right_gripper_visual; collision mesh filename=package://sixdof_pkg/meshes/right_gripper_link.STL scale=1 1 1; visual mesh filename=package://sixdof_pkg/meshes/right_gripper_link.STL scale=1 1 1
- link left_gripper_link: geometry collision mesh filename=package://sixdof_pkg/meshes/left_gripper_link.STL scale=1 1 1; visual mesh filename=package://sixdof_pkg/meshes/left_gripper_link.STL scale=1 1 1
- link right_gripper_link: geometry 
Joints:
- added joint right_gripper_visual_joint: type fixed, parent right_gripper_link, child right_gripper_visual, origin xyz=0 0 0 rpy=3.141592653589793 0 2.8797932657906435
- joint right_gripper: origin xyz=-0.0855 0.0175 0.1025 rpy=-1.5708 0.13911 -1.5708 -> xyz=-0.0855 0.0175 0.1025 rpy=1.570792653589793 3.280703 1.5708
